File: hardware-info/Dyson V6 BMS - PCB 61462 - KiCad Schematic/Dyson V6 BMS - PCB 61462 - KiCad Schematic.kicad_sch (KiCad schematic)
At the start: 118 parts, among them P5 LOAD-, P6 LOAD+, Q1 BC856A, Q2 BC817, Q3 PSMN1R0-30YLC, Q4 PMV45EN, Q5 RTR030N05, U1 PIC16LF1847, U2 ISL94208, U3 MCP1525-TT

Commit message: Schematic Cleanup
Parts:
- removed D3: BAV99, symbol Device:D_Dual_Series_AKC_Parallel
- added D3: BAV99, symbol Device:D_Dual_Series_AKC
Connections:
- net GND: now also D3.2 (K)
- net at R18.1, U2.18 (~{DSENSE}): now also D3.1 (A)
Other:
- note added: "2.5V Ref."
- note added: "Charger/Trigger Detect + Wakeup"
- note added: "VCC Regulation"
- moved on the sheet: C10, C21, C22, C42, C43, C44, C5, C9, D1, D14, D2, D4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

Commit message: Added V7 BMS PCB 279857 Schematic PDF
Other:
- note added: "Adds ability to enable output with series 33R resistor? Why?"
Changed lines of the file:
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@@
     (effects (font (size 1.27 1.27)) (justify left bottom))
   )
-  (text "1C030L" (at 152.4 193.675 0)
+  (text "1C030L" (at 159.385 184.15 0)
     (effects (font (size 1.27 1.27)) (justify left bottom))
   )
@@
     (at 180.34 32.385 0)
     (effects (font (size 0.75 0.75)) (justify right bottom))
+  )
+  (text "Adds ability to enable output\nwith series 33R resistor? Why?"
+    (at 175.26 216.535 0)
+    (effects (font (size 1.27 1.27)) (justify left bottom))
   )
   (label "VPP" (at 375.3034 58.449 0)
@@
   )
   (symbol (lib_id "Device:Fuse") (at 175.895 187.96 270) (mirror x) (unit 1)
-    (in_bom yes) (on_board yes) (fields_autoplaced)
-    (property "Reference" "F1" (id 0) (at 175.895 181.61 90))
-    (property "Value" "30" (id 1) (at 175.895 184.15 90))
+    (in_bom yes) (on_board yes)
+    (property "Reference" "F1" (id 0) (at 176.53 189.865 90))
+    (property "Value" "30" (id 1) (at 176.53 192.405 90))
     (property "Footprint" "" (id 2) (at 175.895 189.738 90)
       (effects (font (size 1.27 1.27)) hide)
